Commit message: Get the stompy running in isaacgym

File: legged_gym/resources/robots/stompypro/robot_fixed.urdf (robot description, URDF)
Before this commit: robot robot, 22 links, 21 joints
Links:
- removed link left_hand_keypoint_link
- removed link right_hand_keypoint_link
- removed link torso_link
- added link base, mass 0.001
Joints:
- removed joint left_hand_keypoint_joint
- removed joint right_hand_keypoint_joint
- removed joint torso_joint
- added joint floating_base: type fixed, parent base, child trunk, origin xyz=0 0 0.0 rpy=0 0 0
- joint L_elbow_x: limit lower=-1.9199 upper=1.9199 effort=17 velocity=5 -> lower=-1.9199 upper=1.9199 effort=17 velocity=0; type revolute -> fixed
- joint L_shoulder_x: limit lower=0 upper=3.1416 effort=60 velocity=5 -> lower=0 upper=3.1416 effort=60 velocity=0; type revolute -> fixed
- joint L_shoulder_y: limit lower=-3.1416 upper=3.1416 effort=60 velocity=5 -> lower=-3.1416 upper=3.1416 effort=60 velocity=0; parent torso_link -> trunk; type revolute -> fixed
- joint L_shoulder_z: limit lower=-3.14 upper=3.14 effort=17 velocity=5 -> lower=-3.14 upper=3.14 effort=17 velocity=0; type revolute -> fixed
- joint R_elbow_x: limit lower=-1.9199 upper=1.9199 effort=17 velocity=5 -> lower=-1.9199 upper=1.9199 effort=17 velocity=0; type revolute -> fixed
- joint R_shoulder_x: limit lower=-3.1416 upper=0 effort=60 velocity=5 -> lower=-3.1416 upper=0 effort=60 velocity=0; type revolute -> fixed
- joint R_shoulder_y: limit lower=-3.1416 upper=3.1416 effort=60 velocity=5 -> lower=-3.1416 upper=3.1416 effort=60 velocity=0; type revolute -> fixed
- joint R_shoulder_z: limit lower=-3.14 upper=3.14 effort=17 velocity=5 -> lower=-3.14 upper=3.14 effort=17 velocity=0; type revolute -> fixed

File: legged_gym/resources/robots/stompypro/robot_test.urdf (robot description, URDF)
Before this commit: robot robot, 22 links, 21 joints
Links:
- removed link left_hand_keypoint_link
- removed link right_hand_keypoint_link
- removed link torso_link
- added link base, mass 0.001
Joints:
- removed joint left_hand_keypoint_joint
- removed joint right_hand_keypoint_joint
- removed joint torso_joint
- added joint floating_base: type fixed, parent base, child trunk, origin xyz=0 0 0.0 rpy=0 0 0
- joint L_shoulder_y: parent torso_link -> trunk
